File: hardware/kicad/bt_resiliency_tester.kicad_pcb (KiCad board)
At the start: 2 copper layers, 96.5 x 73.2 mm, 29 parts, among them J1 UI module, J2 USB-C PWR A, J3 USB-C PWR B, M1 nRF24/E01-2G4M27D, M2 nRF24/E01-2G4M27D, M3 nRF24/E01-2G4M27D, M4 nRF24/E01-2G4M27D, U1 YD-ESP32-23, U2 LD1117V33

Commit message: Add D1 to isolate the devkit's USB power, clearer silkscreen, v0.1 mark
The YD-ESP32-23 passes its USB VBUS out through its 5 V pin, so plugging
the devkit into a PC for programming also powered any E01 radio jumpered
to 5 V on slots 1-2 from the PC port. D1 (1N5819, DO-41) now sits between
+5V_A and the devkit 5 V pin: the USB port feeds only the devkit, and in
battery mode the devkit sees about 4.7 V, fine for its regulator. Radios
still get the full 5 V.

Silkscreen: replace the "RADIO VCC / JPn -> Mn" label with plain wording
(set each radio's jumper: E01 = 5V, NRF24 = 3V3) and add a mirrored
"v0.1" under the goat on the back.

Gerbers, drill files and the fab zip are re-exported with KiCad 10. DRC
has no connection or clearance errors; the six starved-thermal errors at
the radio sockets predate this change. README documents D1.

Co-Authored-By: Claude Fable 5.1 <noreply@anthropic.com>
Parts:
- added D1: 1N5819, Diode_THT:D_DO-41_SOD81_P10.16mm_Horizontal, F.Cu at (62.2, 67.0)
Connections:
- U1 pad 21: +5V_A -> Net-(D1-Pad1)
Routing:
- net Net-(D1-Pad1): track 0.00 -> 6.57 mm
Other:
- board text added: "E01 = 5V"
- board text added: "FOR EACH RADIO"
- board text added: "NRF24 = 3V3"
- board text added: "SET ITS JUMPER:"
- board text added: "v0.1"
- board text removed: "JPn -> Mn"
- board text removed: "RADIO VCC"
