File: hardware/kicad/bt_resiliency_tester.kicad_sch (KiCad schematic)
At the start: 25 parts, among them J1 UI module, J2 USB-C PWR A, J3 USB-C PWR B, M1 nRF24/E01-2G4M27D, M2 nRF24/E01-2G4M27D, M3 nRF24/E01-2G4M27D, M4 nRF24/E01-2G4M27D, U1 YD-ESP32-23, U2 LD1117V33

Commit message: Add D1 to isolate the devkit's USB power, clearer silkscreen, v0.1 mark
The YD-ESP32-23 passes its USB VBUS out through its 5 V pin, so plugging
the devkit into a PC for programming also powered any E01 radio jumpered
to 5 V on slots 1-2 from the PC port. D1 (1N5819, DO-41) now sits between
+5V_A and the devkit 5 V pin: the USB port feeds only the devkit, and in
battery mode the devkit sees about 4.7 V, fine for its regulator. Radios
still get the full 5 V.

Silkscreen: replace the "RADIO VCC / JPn -> Mn" label with plain wording
(set each radio's jumper: E01 = 5V, NRF24 = 3V3) and add a mirrored
"v0.1" under the goat on the back.

Gerbers, drill files and the fab zip are re-exported with KiCad 10. DRC
has no connection or clearance errors; the six starved-thermal errors at
the radio sockets predate this change. README documents D1.

Co-Authored-By: Claude Fable 5.1 <noreply@anthropic.com>
Parts:
- added D1: 1N5819, Diode_THT:D_DO-41_SOD81_P10.16mm_Horizontal, symbol Device:D_Schottky
Connections:
- net +5V_A: now also D1.2 (A); no longer U1.21 (5V)
- new net: D1.1 (K), U1.21 (5V)
Changed lines of the file:
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@@
 		)
 	)
-	(global_label "+5V_A"
-		(at 195.58 173.99 90)
-		(effects
-			(font
-				(size 1.27 1.27)
-			)
-			(justify left)
-		)
-	)
 	(global_label "GND"
 		(at 193.04 247.65 270)
@@
 		)
 	)
+	(symbol
+		(lib_id "Device:D_Schottky")
+		(at 195.58 166.37 90)
+		(unit 1)
+		(body_style 1)
+		(exclude_from_sim no)
+		(in_bom yes)
+		(on_board yes)
+		(in_pos_files yes)
+		(dnp no)
+		(property "Reference" "D1"
+			(at 198.12 166.37 0)
+			(show_name no)
+			(do_not_autoplace no)
+			(effects
+				(font
+					(size 1.27 1.27)
+				)
+			)
+		)
+		(property "Value" "1N5819"
+			(at 193.04 166.37 0)
+			(show_name no)
+			(do_not_autoplace no)
+			(effects
+				(font
+					(size 1.27 1.27)
+				)
+			)
+		)
+		(property "Footprint" "Diode_THT:D_DO-41_SOD81_P10.16mm_Horizontal"
+			(at 195.58 166.37 0)
+			(hide yes)
+			(show_name no)
+			(do_not_autoplace no)
+			(effects
+				(font
+					(size 1.27 1.27)
+				)
+			)
+		)
+		(property "Datasheet" ""
+			(at 195.58 166.37 0)
+			(hide yes)
+			(show_name no)
+			(do_not_autoplace no)
+			(effects
+				(font
+					(size 1.27 1.27)
+				)
+			)
+		)
+		(property "Description" "Schottky diode"
+			(at 195.58 166.37 0)
+			(hide yes)
+			(show_name no)
+			(do_not_autoplace no)
+			(effects
+				(font
+					(size 1.27 1.27)
+				)
+			)
+		)
+		(pin "1"
+		)
+		(pin "2"
+		)
+		(instances
+			(project "bt_resiliency_tester"
+				(path "/759d86e3-0625-40b8-a3e4-c4e2bfc9e187"
+					(reference "D1")
+					(unit 1)
+				)
+			)
+		)
+	)
+	(wire
+		(pts
+			(xy 195.58 170.18) (xy 195.57999999999998 173.99)
+		)
+		(stroke
+			(width 0)
+			(type default)
+		)
+	)
+	(global_label "+5V_A"
+		(at 195.58 162.56 90)
+		(effects
+			(font
+				(size 1.27 1.27)
+			)
+			(justify left)
+		)
+	)
