File: hardware/kicad/bt_radio_manager.kicad_pcb (KiCad board)
At the start: 2 copper layers, 96.5 x 73.2 mm, 30 parts, among them J1 UI module, J2 USB-C PWR A, J3 USB-C PWR B, M1 nRF24/E01-2G4M27D, M2 nRF24/E01-2G4M27D, M3 nRF24/E01-2G4M27D, M4 nRF24/E01-2G4M27D, U1 YD-ESP32-23, U2 LD1117V33

Commit message: Power: D2/D3 cross-feed so one 5V supply or two both work, v0.2
Two SB240 Schottkys (DO-15) join +5V_A and +5V_B in opposite
directions. With two supplies each rail runs from its own input; with
one (preferably J2) the other rail is fed through a diode. The 5V
power traces, previously 0.2 mm, are re-routed at 0.6-1.0 mm for the
~1.9 A single-supply case. Diodes placed clear of the USB-C socket
bodies (case clearance check passes for both radio variants).

Both board variants updated, gerbers and order zip re-exported,
README power section and BOM updated, version mark bumped to v0.2.

Co-Authored-By: Claude Opus 5.5 <noreply@anthropic.com>
Parts:
- added D2: SB240, Diode_THT:D_DO-15_P10.16mm_Horizontal, F.Cu at (22.3, 63.6)
- added D3: SB240, Diode_THT:D_DO-15_P10.16mm_Horizontal, F.Cu at (32.5, 58.6)
Routing:
- net +5V_B: track 61.3 -> 74.1 mm
- net +5V_A: track 69.6 -> 66.3 mm
Other:
- board text added: "1 SUPPLY: J2"
- board text added: "v0.2"
- board text removed: "v0.1"
